File: pcbs/phantoma/phantoma.kicad_pcb (KiCad board)
At the start: 2 copper layers, 118.1 x 90.3 mm, 19 parts, among them SW1 SW_PUSH, SW10 SW_PUSH, SW11 SW_PUSH, SW12 SW_PUSH, SW13 SW_PUSH, SW14 SW_PUSH, SW15 SW_PUSH, SW2 SW_PUSH, SW3 SW_PUSH, SW4 SW_PUSH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

Commit message: oopsies
Routing:
- net GND: track 350.6 -> 349.6 mm
