File: pcbs/phantoma/phantoma.kicad_pcb (KiCad board)
At the start: 2 copper layers, 118.1 x 90.3 mm, 19 parts, among them SW1 SW_PUSH, SW10 SW_PUSH, SW11 SW_PUSH, SW12 SW_PUSH, SW13 SW_PUSH, SW14 SW_PUSH, SW15 SW_PUSH, SW2 SW_PUSH, SW3 SW_PUSH, SW4 SW_PUSH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

Commit message: lotsa changes
Parts:
- removed REF**: Tenting Puck, kbd:Tenting_Puck2
Other:
- board text added: "ファントマ"
- board text removed: "<3 ファントマ"

Commit message: added reset footprint and generally outchea makin' changes
Parts:
- added SW16: SW_Push, kbd:ResetSW, F.Cu at (112.1, 45.5)
Connections:
- U1 pad 22: unconnected-(U1-Pad22) -> reset
Routing:
- net reset: track 0.00 -> 53.8 mm, vias 0 -> 1
- net GND: track 349.6 -> 381.2 mm
- net unconnected-(U1-Pad22): track 12.5 -> 0.00 mm, vias 1 -> 0
