File: pcbs/artemis/artemis.kicad_sch (KiCad schematic)
At the start: 20 parts, among them SW1 SW_PUSH, SW10 SW_PUSH, SW11 SW_PUSH, SW12 SW_PUSH, SW13 SW_PUSH, SW14 SW_PUSH, SW15 SW_PUSH, SW16 SW_PUSH, SW17 SW_PUSH, SW2 SW_PUSH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

Commit message: added reset footprint and generally outchea makin' changes
Parts:
- added SW18: SW_Push, kbd:ResetSW, symbol Switch:SW_Push
Connections:
- net reset: now reaches U1.22 (RST)
- net reset: now also SW18.1
- new net gnd: SW18.2
- no-connect marks 3 -> 2
Changed lines of the file:
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@@
   (title_block
     (title "artemis (アルテミス)")
-    (date "2022-01-08")
-    (rev "0.2")
+    (date "2022-01-25")
+    (rev "0.3")
     (company "<3")
   )
@@
   (no_connect (at 118.11 52.07))
   (no_connect (at 41.91 36.83))
-  (no_connect (at 77.47 39.37))
   (wire (pts (xy 41.91 39.37) (xy 41.91 41.91))
     (stroke (width 0) (type solid) (color 0 0 0 0))
+  )
+  (global_label "reset" (shape input) (at 77.47 39.37 0) (fields_autoplaced)
+    (effects (font (size 1.27 1.27)) (justify left))
+    (property "Intersheet References" "${INTERSHEET_REFS}" (id 0) (at 84.5113 39.2906 0)
+      (effects (font (size 1.27 1.27)) (justify left) hide)
+    )
   )
   (global_label "switch4" (shape input) (at 77.47 59.69 0) (fields_autoplaced)
@@
     )
   )
+  (global_label "gnd" (shape input) (at 106.68 50.8 0) (fields_autoplaced)
+    (effects (font (size 1.27 1.27)) (justify left))
+    (property "Intersheet References" "${INTERSHEET_REFS}" (id 0) (at 112.4005 50.7206 0)
+      (effects (font (size 1.27 1.27)) (justify left) hide)
+    )
+  )
   (global_label "switch17" (shape input) (at 120.65 123.19 90) (fields_autoplaced)
     (effects (font (size 1.27 1.27)) (justify left))
@@
     (effects (font (size 1.27 1.27)) (justify right))
     (property "Intersheet References" "${INTERSHEET_REFS}" (id 0) (at 31.2401 54.5306 0)
+      (effects (font (size 1.27 1.27)) (justify right) hide)
+    )
+  )
+  (global_label "reset" (shape input) (at 96.52 50.8 180) (fields_autoplaced)
+    (effects (font (size 1.27 1.27)) (justify right))
+    (property "Intersheet References" "${INTERSHEET_REFS}" (id 0) (at 89.5295 50.7206 0)
       (effects (font (size 1.27 1.27)) (justify right) hide)
     )
@@
     (pin "1")
   )
+  (symbol (lib_id "Switch:SW_Push") (at 101.6 50.8 0) (unit 1)
+    (in_bom yes) (on_board yes) (fields_autoplaced)
+    (property "Reference" "SW18" (id 0) (at 101.6 43.18 0))
+    (property "Value" "SW_Push" (id 1) (at 101.6 45.72 0))
+    (property "Footprint" "kbd:ResetSW" (id 2) (at 101.6 45.72 0)
+      (effects (font (size 1.27 1.27)) hide)
+    )
+    (property "Datasheet" "~" (id 3) (at 101.6 45.72 0)
+      (effects (font (size 1.27 1.27)) hide)
+    )
+    (pin "1")
+    (pin "2")
+  )
   (symbol (lib_id "power:GND") (at 95.25 110.49 0) (unit 1)
     (in_bom yes) (on_board yes) (fields_autoplaced)
@@
       (reference "SW17") (unit 1) (value "SW_PUSH") (footprint "bugs:Choc_reversible")
     )
+    (path "/32f4eb0d-8b7c-4e0f-8b4a-904219172497"
+      (reference "SW18") (unit 1) (value "SW_Push") (footprint "kbd:ResetSW")
+    )
     (path "/00000000-0000-0000-0000-00005a5e14c2"
