File: pcbs/luna/luna.kicad_pcb (KiCad board)
At the start: 2 copper layers, 116.9 x 79.4 mm, 20 parts, among them SW1 SW_PUSH, SW10 SW_PUSH, SW11 SW_PUSH, SW12 SW_PUSH, SW13 SW_PUSH, SW14 SW_PUSH, SW15 SW_PUSH, SW2 SW_PUSH, SW3 SW_PUSH, SW4 SW_PUSH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

Commit message: added reset footprint and generally outchea makin' changes
Parts:
- added SW16: SW_Push, kbd:ResetSW, F.Cu at (111.5, 58.2)
- SW1, SW10, SW11, SW12, SW13, SW2, SW3, SW4, SW5, SW6, SW7, SW8, SW9: footprint bugs:Choc_reversible -> bugs:Kailh_socket_PG1350_optional_reversible_1u
- SW14, SW15: footprint bugs:Choc_reversible_15u -> bugs:Kailh_socket_PG1350_optional_reversible_15u
- moved BT1 25.4 mm to (140.1, 95.6), turned to -90 degrees
- moved SW14 0.16 mm to (105.9, 113.5)
- moved SW15 0.15 mm to (128.2, 110.7)
Connections:
- SW1 pad 1: switch1 -> GND
- SW12 pad 2: GND -> switch12
- SW13 pad 1: switch13 -> GND
- SW13 pad 2: GND -> switch13
- SW14 pad 1: switch14 -> GND
- SW3 pad 1: switch3 -> GND
- SW5 pad 1: switch5 -> GND
- SW6 pad 2: GND -> switch6
- SW8 pad 1: switch8 -> GND
- SW9 pad 2: GND -> switch9
- U1 pad 14: switch10 -> switch4
- U1 pad 15: switch4 -> switch3
- U1 pad 16: switch3 -> switch2
- U1 pad 17: switch2 -> switch10
- U1 pad 22: unconnected-(U1-Pad22) -> reset
Routing:
- net GND: track 347.2 -> 743.6 mm
- net switch15: track 42.5 -> 86.1 mm
- net reset: track 0.00 -> 42.3 mm, vias 0 -> 1
- net Net-(BT1-Pad2): track 12.1 -> 44.7 mm, vias 2 -> 3
- net switch10: track 39.0 -> 71.4 mm
- net raw: track 17.2 -> 46.0 mm, vias 3 -> 4
- net switch1: track 147.7 -> 171.3 mm
- net switch11: track 107.1 -> 130.6 mm
- net switch12: track 91.4 -> 114.8 mm
- net switch13: track 72.0 -> 95.1 mm
- net switch6: track 127.3 -> 148.8 mm
- net switch8: track 99.0 -> 120.4 mm
- net switch5: track 52.2 -> 73.4 mm
- net switch14: track 70.2 -> 91.3 mm
- net switch7: track 120.3 -> 140.9 mm
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Other:
- board size 116.9 x 79.4 mm -> 118.1 x 79.5 mm
