File: pcbs/luna/luna.kicad_sch (KiCad schematic)
At the start: 18 parts, among them SW1 SW_PUSH, SW10 SW_PUSH, SW11 SW_PUSH, SW12 SW_PUSH, SW13 SW_PUSH, SW14 SW_PUSH, SW15 SW_PUSH, SW2 SW_PUSH, SW3 SW_PUSH, SW4 SW_PUSH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

Commit message: added reset footprint and generally outchea makin' changes
Parts:
- added SW16: SW_Push, kbd:ResetSW, symbol Switch:SW_Push
Connections:
- net switch10: now also U1.17 (F7); no longer U1.14 (B2)
- net switch2: now also U1.16 (B1); no longer U1.17 (F7)
- net switch3: now also U1.15 (B3); no longer U1.16 (B1)
- net switch4: now also U1.14 (B2); no longer U1.15 (B3)
- net reset: now reaches U1.22 (RST)
- net reset: now also SW16.1
- new net gnd: SW16.2
- no-connect marks 5 -> 4
Changed lines of the file:
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@@
   (title_block
     (title "luna (ルナ)")
-    (date "2022-01-08")
-    (rev "0.2")
+    (date "2022-01-25")
+    (rev "0.3")
     (company "<3")
   )
@@
   (no_connect (at 41.91 36.83))
   (no_connect (at 77.47 44.45))
-  (no_connect (at 77.47 39.37))
   (wire (pts (xy 41.91 39.37) (xy 41.91 41.91))
     (stroke (width 0) (type solid) (color 0 0 0 0))
   )
-  (global_label "switch4" (shape input) (at 77.47 57.15 0) (fields_autoplaced)
+  (global_label "reset" (shape input) (at 77.47 39.37 0) (fields_autoplaced)
+    (effects (font (size 1.27 1.27)) (justify left))
+    (property "Intersheet References" "${INTERSHEET_REFS}" (id 0) (at 84.5113 39.2906 0)
+      (effects (font (size 1.27 1.27)) (justify left) hide)
+    )
+  )
+  (global_label "switch3" (shape input) (at 77.47 57.15 0) (fields_autoplaced)
     (effects (font (size 1.27 1.27)) (justify left))
     (property "Intersheet References" "${INTERSHEET_REFS}" (id 0) (at 86.9304 57.0706 0)
@@
     )
   )
+  (global_label "gnd" (shape input) (at 107.95 52.07 0) (fields_autoplaced)
+    (effects (font (size 1.27 1.27)) (justify left))
+    (property "Intersheet References" "${INTERSHEET_REFS}" (id 0) (at 113.6705 51.9906 0)
+      (effects (font (size 1.27 1.27)) (justify left) hide)
+    )
+  )
   (global_label "switch7" (shape input) (at 59.69 97.79 90) (fields_autoplaced)
     (effects (font (size 1.27 1.27)) (justify left))
@@
     )
   )
-  (global_label "switch10" (shape input) (at 77.47 59.69 0) (fields_autoplaced)
-    (effects (font (size 1.27 1.27)) (justify left))
-    (property "Intersheet References" "${INTERSHEET_REFS}" (id 0) (at 88.1399 59.6106 0)
+  (global_label "switch4" (shape input) (at 77.47 59.69 0) (fields_autoplaced)
+    (effects (font (size 1.27 1.27)) (justify left))
+    (property "Intersheet References" "${INTERSHEET_REFS}" (id 0) (at 86.9304 59.6106 0)
       (effects (font (size 1.27 1.27)) (justify left) hide)
     )
@@
     (property "Intersheet References" "${INTERSHEET_REFS}" (id 0) (at 83.0091 34.2106 0)
       (effects (font (size 1.27 1.27)) (justify left) hide)
+    )
+  )
+  (global_label "reset" (shape input) (at 97.79 52.07 180) (fields_autoplaced)
+    (effects (font (size 1.27 1.27)) (justify right))
+    (property "Intersheet References" "${INTERSHEET_REFS}" (id 0) (at 90.7995 51.9906 0)
+      (effects (font (size 1.27 1.27)) (justify right) hide)
     )
   )
@@
     )
   )
-  (global_label "switch3" (shape input) (at 77.47 54.61 0) (fields_autoplaced)
+  (global_label "switch2" (shape input) (at 77.47 54.61 0) (fields_autoplaced)
     (effects (font (size 1.27 1.27)) (justify left))
     (property "Intersheet References" "${INTERSHEET_REFS}" (id 0) (at 86.9304 54.5306 0)
@@
     )
   )
-  (global_label "switch2" (shape input) (at 77.47 52.07 0) (fields_autoplaced)
-    (effects (font (size 1.27 1.27)) (justify left))
-    (property "Intersheet References" "${INTERSHEET_REFS}" (id 0) (at 86.9304 51.9906 0)
+  (global_label "switch10" (shape input) (at 77.47 52.07 0) (fields_autoplaced)
+    (effects (font (size 1.27 1.27)) (justify left))
+    (property "Intersheet References" "${INTERSHEET_REFS}" (id 0) (at 88.1399 51.9906 0)
       (effects (font (size 1.27 1.27)) (justify left) hide)
     )
@@
     (pin "1")
   )
+  (symbol (lib_id "Switch:SW_Push") (at 102.87 52.07 0) (unit 1)
+    (in_bom yes) (on_board yes) (fields_autoplaced)
+    (property "Reference" "SW16" (id 0) (at 102.87 44.45 0))
+    (property "Value" "SW_Push" (id 1) (at 102.87 46.99 0))
+    (property "Footprint" "kbd:ResetSW" (id 2) (at 102.87 46.99 0)
+      (effects (font (size 1.27 1.27)) hide)
+    )
+    (property "Datasheet" "~" (id 3) (at 102.87 46.99 0)
+      (effects (font (size 1.27 1.27)) hide)
+    )
+    (pin "1")
+    (pin "2")
+  )
   (symbol (lib_id "power:GND") (at 74.93 85.09 0) (unit 1)
     (in_bom yes) (on_board yes) (fields_autoplaced)
@@
       (reference "SW15") (unit 1) (value "SW_PUSH") (footprint "bugs:Choc_reversible")
     )
+    (path "/be40a792-1fff-4ce1-a6d8-41730132bad4"
+      (reference "SW16") (unit 1) (value "SW_Push") (footprint "kbd:ResetSW")
+    )
     (path "/00000000-0000-0000-0000-00005a5e14c2"
