File: pcbs/minako/minako.kicad_sch (KiCad schematic)
At the start: 19 parts, among them SW1 SW_PUSH, SW10 SW_PUSH, SW11 SW_PUSH, SW12 SW_PUSH, SW13 SW_PUSH, SW14 SW_PUSH, SW15 SW_PUSH, SW16 SW_PUSH, SW2 SW_PUSH, SW3 SW_PUSH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

Commit message: added reset footprint and generally outchea makin' changes
Parts:
- added SW17: SW_Push, kbd:ResetSW, symbol Switch:SW_Push
Connections:
- net reset: now reaches U1.22 (RST)
- net reset: now also SW17.1
- new net gnd: SW17.2
- no-connect marks 4 -> 3
Changed lines of the file:
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@@
   (title_block
     (title "minako (美奈子)")
-    (date "2022-01-08")
-    (rev "0.2")
+    (date "2022-01-25")
+    (rev "0.3")
     (company "<3")
   )
@@
   (no_connect (at 41.91 36.83))
   (no_connect (at 41.91 34.29))
-  (no_connect (at 77.47 39.37))
   (wire (pts (xy 41.91 39.37) (xy 41.91 41.91))
     (stroke (width 0) (type solid) (color 0 0 0 0))
@@
     )
   )
+  (global_label "reset" (shape input) (at 97.79 52.07 180) (fields_autoplaced)
+    (effects (font (size 1.27 1.27)) (justify right))
+    (property "Intersheet References" "${INTERSHEET_REFS}" (id 0) (at 90.7995 51.9906 0)
+      (effects (font (size 1.27 1.27)) (justify right) hide)
+    )
+  )
   (global_label "switch9" (shape input) (at 77.47 46.99 0) (fields_autoplaced)
     (effects (font (size 1.27 1.27)) (justify left))
@@
     )
   )
+  (global_label "reset" (shape input) (at 77.47 39.37 0) (fields_autoplaced)
+    (effects (font (size 1.27 1.27)) (justify left))
+    (property "Intersheet References" "${INTERSHEET_REFS}" (id 0) (at 84.5113 39.2906 0)
+      (effects (font (size 1.27 1.27)) (justify left) hide)
+    )
+  )
   (global_label "switch6" (shape input) (at 34.29 105.41 90) (fields_autoplaced)
     (effects (font (size 1.27 1.27)) (justify left))
@@
     (effects (font (size 1.27 1.27)) (justify left))
     (property "Intersheet References" "${INTERSHEET_REFS}" (id 0) (at 88.2288 62.1506 0)
+      (effects (font (size 1.27 1.27)) (justify left) hide)
+    )
+  )
+  (global_label "gnd" (shape input) (at 107.95 52.07 0) (fields_autoplaced)
+    (effects (font (size 1.27 1.27)) (justify left))
+    (property "Intersheet References" "${INTERSHEET_REFS}" (id 0) (at 113.6705 51.9906 0)
       (effects (font (size 1.27 1.27)) (justify left) hide)
     )
@@
     (pin "1")
   )
+  (symbol (lib_id "Switch:SW_Push") (at 102.87 52.07 0) (unit 1)
+    (in_bom yes) (on_board yes) (fields_autoplaced)
+    (property "Reference" "SW17" (id 0) (at 102.87 44.45 0))
+    (property "Value" "SW_Push" (id 1) (at 102.87 46.99 0))
+    (property "Footprint" "kbd:ResetSW" (id 2) (at 102.87 46.99 0)
+      (effects (font (size 1.27 1.27)) hide)
+    )
+    (property "Datasheet" "~" (id 3) (at 102.87 46.99 0)
+      (effects (font (size 1.27 1.27)) hide)
+    )
+    (pin "1")
+    (pin "2")
+  )
   (symbol (lib_id "power:GND") (at 110.49 132.08 0) (unit 1)
     (in_bom yes) (on_board yes) (fields_autoplaced)
@@
       (reference "SW16") (unit 1) (value "SW_PUSH") (footprint "bugs:Choc_reversible")
     )
+    (path "/c66790a8-2c84-47da-b059-a728d9f51463"
+      (reference "SW17") (unit 1) (value "SW_Push") (footprint "kbd:ResetSW")
+    )
     (path "/00000000-0000-0000-0000-00005a5e14c2"
